File: circuits/PRE/preDiff.sch (KiCad schematic (older format))
At the start: 46 parts, among them K1 CONN_3, P1 CONN_1, P2 CONN_1, P3 CONN_1, P4 CONN_1, P5 CONN_1, P6 CONN_1, P7 CONN_1, P8 CONN_1, P9 CONN_1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

Commit message: revisado entrada pre
Parts:
- removed C7: 100p, symbol C
- added C13, C14, C15, C7: CP, symbol CP
- added C16: 100p, symbol C
- added P10: CONN_1, symbol CONN_1
- added R17: 6k8, symbol R
- added R18: R, symbol R
- R1, R4: value R -> 10
- R5: value R -> 6k8
Connections:
- net GND: now also C16.2, R18.1; no longer R1.1
- net at C1.1, D6.2 (K), U1.5 (+): now also D2.1 (A), D4.2 (K), R3.1, R4.2; no longer R5.2
- net at C1.2, D5.2 (K), U1.3 (+): now also D1.1 (A), D3.2 (K), R1.2, R2.2; no longer R4.2
- net at R2.1, R3.2: now also R18.2; no longer R1.2
- net at C5.2, K1.2 (PM), P2.1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: now also R17.1
- net at C4.1, K1.3 (P3), P1.1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: now also R5.1
- net at C4.2, C5.1: now also C16.1
- net at C6.1, P8.1, R14.2: now also C14.1, C15.1
- net at C8.1, P9.1, R15.2: now also C13.1, C7.1
- new net: C13.2, C7.2, C8.2, R4.1
- new net: C14.2, C15.2, C6.2, R1.1
- new net: P10.1, R17.2, R5.2
Other:
- moved on the sheet: C1, C10, C11, C12, C2, C3, C4, C5, C6, C8, C9, D1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

Commit message: input from pre separated
Parts:
- added C?: CP, symbol CP
- added P11: CONN_1, symbol CONN_1
- added R19: 47k, symbol R
Connections:
- net GND: now also C?.2, R19.2
- net at P10.1, R17.2, R5.2: now also C?.1
- new net: P11.1, R19.1
Changed lines of the file:
@@
-EESchema Schematic File Version 2  date Sat 02 Apr 2016 01:04:31 PM ART
+EESchema Schematic File Version 2  date Sat 02 Apr 2016 03:19:25 PM ART
 LIBS:power
 LIBS:device
@@
 Comment4 ""
 $EndDescr
-$Comp
-L C C16
-U 1 1 56FFED60
-P 1950 3300
-F 0 "C16" H 2000 3400 50  0000 L CNN
-F 1 "100p" H 2000 3200 50  0000 L CNN
-	1    1950 3300
-	0    -1   -1   0
-$EndComp
-$Comp
-L R R18
-U 1 1 56FFED58
-P 4800 3300
-F 0 "R18" V 4880 3300 50  0000 C CNN
-F 1 "R" V 4800 3300 50  0000 C CNN
-	1    4800 3300
-	0    -1   -1   0
-$EndComp
+Wire Wire Line
+	1400 1200 1400 1800
 Connection ~ 5300 2700
 Connection ~ 5300 3850
-$Comp
-L CONN_1 P10
-U 1 1 56FFECEC
-P 1550 1650
-F 0 "P10" H 1630 1650 40  0000 L CNN
-F 1 "CONN_1" H 1550 1705 30  0001 C CNN
-	1    1550 1650
-	0    -1   -1   0
-$EndComp
 Connection ~ 1400 2500
 Wire Wire Line
@@
 Wire Wire Line
 	1400 1800 1550 1800
+Wire Wire Line
+	1800 1200 2450 1200
+Wire Wire Line
+	2450 1200 2450 1900
+Connection ~ 2450 1800
+$Comp
+L CP C?
+U 1 1 56FFF540
+P 1600 1200
+F 0 "C?" H 1650 1300 50  0000 L CNN
+F 1 "CP" H 1650 1100 50  0000 L CNN
+	1    1600 1200
+	0    -1   -1   0
+$EndComp
+$Comp
+L GND #PWR01
+U 1 1 56FFF2B7
+P 2450 1900
+F 0 "#PWR01" H 2450 1900 30  0001 C CNN
+F 1 "GND" H 2450 1830 30  0001 C CNN
+	1    2450 1900
+	1    0    0    -1
+$EndComp
+$Comp
+L R R19
+U 1 1 56FFF2A8
+P 2200 1800
+F 0 "R19" V 2280 1800 50  0000 C CNN
+F 1 "47k" V 2200 1800 50  0000 C CNN
+	1    2200 1800
+	0    -1   -1   0
+$EndComp
+$Comp
+L CONN_1 P11
+U 1 1 56FFF2A2
+P 1950 1650
+F 0 "P11" H 2030 1650 40  0000 L CNN
+F 1 "CONN_1" H 1950 1705 30  0001 C CNN
+	1    1950 1650
+	0    -1   -1   0
+$EndComp
+$Comp
+L C C16
+U 1 1 56FFED60
+P 1950 3300
+F 0 "C16" H 2000 3400 50  0000 L CNN
+F 1 "100p" H 2000 3200 50  0000 L CNN
+	1    1950 3300
+	0    -1   -1   0
+$EndComp
+$Comp
+L R R18
+U 1 1 56FFED58
+P 4800 3300
+F 0 "R18" V 4880 3300 50  0000 C CNN
+F 1 "R" V 4800 3300 50  0000 C CNN
+	1    4800 3300
+	0    -1   -1   0
+$EndComp
+$Comp
+L CONN_1 P10
+U 1 1 56FFECEC
+P 1550 1650
+F 0 "P10" H 1630 1650 40  0000 L CNN
+F 1 "CONN_1" H 1550 1705 30  0001 C CNN
+	1    1550 1650
+	0    -1   -1   0
+$EndComp
 $Comp
 L R R5
@@
 $EndComp
 $Comp
-L GND #PWR01
+L GND #PWR02
 U 1 1 56FE9B52
 P 4250 3450
-F 0 "#PWR01" H 4250 3450 30  0001 C CNN
+F 0 "#PWR02" H 4250 3450 30  0001 C CNN
 F 1 "GND" H 4250 3380 30  0001 C CNN
 	1    4250 3450
@@
 $EndComp
 $Comp
-L GND #PWR02
+L GND #PWR03
 U 1 1 56FE9B25
 P 3700 3550
-F 0 "#PWR02" H 3700 3550 30  0001 C CNN
+F 0 "#PWR03" H 3700 3550 30  0001 C CNN
 F 1 "GND" H 3700 3480 30  0001 C CNN
 	1    3700 3550
@@
 $EndComp
 $Comp
-L GND #PWR03
+L GND #PWR04
 U 1 1 56FE993D
 P 9900 2400
-F 0 "#PWR03" H 9900 2400 30  0001 C CNN
+F 0 "#PWR04" H 9900 2400 30  0001 C CNN
 F 1 "GND" H 9900 2330 30  0001 C CNN
 	1    9900 2400
@@
 $EndComp
 $Comp
-L GND #PWR04
+L GND #PWR05
 U 1 1 56FE9938
 P 8400 2300
-F 0 "#PWR04" H 8400 2300 30  0001 C CNN
+F 0 "#PWR05" H 8400 2300 30  0001 C CNN
 F 1 "GND" H 8400 2230 30  0001 C CNN
 	1    8400 2300
@@
 $EndComp
 $Comp
-L GND #PWR05
+L GND #PWR06
 U 1 1 56FE97E8
 P 2150 3500
-F 0 "#PWR05" H 2150 3500 30  0001 C CNN
+F 0 "#PWR06" H 2150 3500 30  0001 C CNN
 F 1 "GND" H 2150 3430 30  0001 C CNN
 	1    2150 3500
@@
 $EndComp
 $Comp
-L GND #PWR06
+L GND #PWR07
 U 1 1 56FE97A7
 P 1400 3500
-F 0 "#PWR06" H 1400 3500 30  0001 C CNN
+F 0 "#PWR07" H 1400 3500 30  0001 C CNN
 F 1 "GND" H 1400 3430 30  0001 C CNN
 	1    1400 3500
@@
 $EndComp
 $Comp
-L VCC #PWR07
+L VCC #PWR08
 U 1 1 56FE9547
 P 4050 3300
-F 0 "#PWR07" H 4050 3400 30  0001 C CNN
+F 0 "#PWR08" H 4050 3400 30  0001 C CNN
 F 1 "VCC" H 4050 3400 30  0000 C CNN
 	1    4050 3300
@@
 $EndComp
 $Comp
-L VDD #PWR08
+L VDD #PWR09
 U 1 1 56FE9539
 P 4450 3300
-F 0 "#PWR08" H 4450 3400 30  0001 C CNN
+F 0 "#PWR09" H 4450 3400 30  0001 C CNN
 F 1 "VDD" H 4450 3410 30  0000 C CNN
 	1    4450 3300
@@
 $EndComp
 $Comp
-L PWR_FLAG #FLG09
+L PWR_FLAG #FLG010
 U 1 1 56FE8A32
 P 9500 2300
-F 0 "#FLG09" H 9500 2395 30  0001 C CNN
+F 0 "#FLG010" H 9500 2395 30  0001 C CNN
 F 1 "PWR_FLAG" H 9500 2480 30  0000 C CNN
 	1    9500 2300
@@
 $EndComp
 $Comp
-L PWR_FLAG #FLG010
+L PWR_FLAG #FLG011
 U 1 1 56FE8A22
 P 8000 2200
-F 0 "#FLG010" H 8000 2295 30  0001 C CNN
+F 0 "#FLG011" H 8000 2295 30  0001 C CNN
 F 1 "PWR_FLAG" H 8000 2380 30  0000 C CNN
 	1    8000 2200
@@
 $EndComp
 $Comp
-L PWR_FLAG #FLG011
+L PWR_FLAG #FLG012
 U 1 1 56FE8A19
 P 4550 3300
-F 0 "#FLG011" H 4550 3395 30  0001 C CNN
+F 0 "#FLG012" H 4550 3395 30  0001 C CNN
 F 1 "PWR_FLAG" H 4550 3480 30  0000 C CNN
 	1    4550 3300
@@
 $EndComp
 $Comp
-L GND #PWR012
+L GND #PWR013
 U 1 1 56FE89F6
 P 4550 3450
-F 0 "#PWR012" H 4550 3450 30  0001 C CNN
+F 0 "#PWR013" H 4550 3450 30  0001 C CNN
 F 1 "GND" H 4550 3380 30  0001 C CNN
 	1    4550 3450
@@
 $EndComp
 $Comp
-L GND #PWR013
+L GND #PWR014
 U 1 1 56FE89D1
 P 10600 4200
-F 0 "#PWR013" H 10600 4200 30  0001 C CNN
+F 0 "#PWR014" H 10600 4200 30  0001 C CNN
 F 1 "GND" H 10600 4130 30  0001 C CNN
 	1    10600 4200
@@
 $EndComp
 $Comp
-L VDD #PWR014
+L VDD #PWR015
 U 1 1 56FE7200
 P 9500 2300
-F 0 "#PWR014" H 9500 2400 30  0001 C CNN
+F 0 "#PWR015" H 9500 2400 30  0001 C CNN
 F 1 "VDD" H 9500 2410 30  0000 C CNN
 	1    9500 2300
@@
 $EndComp
 $Comp
-L VCC #PWR015
+L VCC #PWR016
 U 1 1 56FE70C7
 P 8000 2200
-F 0 "#PWR015" H 8000 2300 30  0001 C CNN
+F 0 "#PWR016" H 8000 2300 30  0001 C CNN
 F 1 "VCC" H 8000 2300 30  0000 C CNN
 	1    8000 2200
